File: pcb/mcu.kicad_sch (KiCad schematic)
At the start: 3 parts, among them U3 ATtiny1616-M

Commit message: rev0 done
Connections:
- net DRV_nSHDN: now reaches U3.5 (PA4)
- net EN_LED: no longer names the net of U3.14 (PB0)
Changed lines of the file:
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@@
+	)
+	(no_connect
+		(at 148.59 96.52)
 	)
 	(no_connect
 		(at 148.59 86.36)
-	)
-	(no_connect
-		(at 148.59 83.82)
 	)
 	(no_connect
@@
 		)
 	)
-	(hierarchical_label "EN_LED"
+	(hierarchical_label "DRV_nSHDN"
 		(shape output)
-		(at 148.59 96.52 0)
-		(effects
-			(font
+		(at 148.59 83.82 0)
+		(effects
+			(font
