File: pcb/lightwear.kicad_pcb (KiCad board)
At the start: 2 copper layers, 55 x 20 mm, 2 parts, among them J1 USB_C_Receptacle_USB2.0_16P

Commit message: rev0 done
Parts:
- added C1: 100nF, Capacitor_SMD:C_0402_1005Metric, F.Cu at (168.8, 54.9)
- added C2: 1uF 35V, Capacitor_SMD:C_0603_1608Metric, F.Cu at (165.6, 61.4)
- added C4: 100nF, Capacitor_SMD:C_0402_1005Metric, F.Cu at (158.8, 64.0)
- added C5: 2.2uF, Capacitor_SMD:C_0402_1005Metric, F.Cu at (158.8, 65.1)
- added C6: 470nF, Capacitor_SMD:C_0402_1005Metric, F.Cu at (148.9, 64.8)
- added C7: 4.7uF, Capacitor_SMD:C_0402_1005Metric, F.Cu at (170.7, 54.9)
- added C8: 1uF 30V, Capacitor_SMD:C_0402_1005Metric, F.Cu at (160.2, 55.2)
- added D1: D_Schottky 30V, Diode_SMD:D_SOD-123, F.Cu at (165.6, 59.5)
- added L1: 4.7uH, Inductor_SMD:L_Changjiang_FNR4030S, B.Cu at (173.0, 55.3)
- added Q1: PMOS, Package_TO_SOT_SMD:SOT-23-3, F.Cu at (158.1, 59.1)
- added R1: 33R, Resistor_SMD:R_0402_1005Metric, F.Cu at (148.9, 63.7)
- added R10: 200k 30V, Resistor_SMD:R_0402_1005Metric, F.Cu at (161.3, 55.2)
- added R11: 5.1k, Resistor_SMD:R_0402_1005Metric, F.Cu at (158.8, 62.9)
- added R12: 10k 30V, Resistor_SMD:R_0402_1005Metric, F.Cu at (162.4, 55.2)
- added R3: 5.1k, Resistor_SMD:R_0402_1005Metric, F.Cu at (173.7, 62.4)
- added R4: 5.1k, Resistor_SMD:R_0402_1005Metric, F.Cu at (173.7, 64.4)
- added R6: 0.05R, Resistor_SMD:R_1206_3216Metric, F.Cu at (165.5, 64.6)
- added R7: 100k 30V, Resistor_SMD:R_0402_1005Metric, F.Cu at (158.8, 61.8)
- added R8: 2k, Resistor_SMD:R_0402_1005Metric, F.Cu at (159.1, 55.2)
- added R9: 0R, Resistor_SMD:R_0402_1005Metric, F.Cu at (155.0, 61.6)
- added SW1: SW_SPST, footprints:SW4_PTS815 SJM 250 SMTR LFS_CNK, F.Cu at (140.2, 62.8)
- added TP1: USB_SBU1, TestPoint:TestPoint_Pad_D2.0mm, F.Cu at (147.7, 61.3)
- added TP10: PA2, TestPoint:TestPoint_Pad_D2.0mm, F.Cu at (136.2, 68.5)
- added TP11: PB2, TestPoint:TestPoint_Pad_D2.0mm, F.Cu at (138.8, 56.2)
- added TP12: PB3, TestPoint:TestPoint_Pad_D2.0mm, F.Cu at (135.3, 56.2)
- added TP13: PC1, TestPoint:TestPoint_Pad_D2.0mm, F.Cu at (132.7, 68.5)
- added TP14: PC2, TestPoint:TestPoint_Pad_D2.0mm, F.Cu at (129.2, 68.5)
- added TP16: USB_SBU2, TestPoint:TestPoint_Pad_D2.0mm, F.Cu at (150.9, 58.5)
- added TP2: BTN, TestPoint:TestPoint_Pad_D2.0mm, F.Cu at (147.1, 67.2)
- added TP3: MCU_VCC, TestPoint:TestPoint_Pad_D1.5mm, F.Cu at (157.2, 69.9)
- added TP4: UPDI, TestPoint:TestPoint_Pad_D1.5mm, F.Cu at (154.8, 69.9)
- added TP5: GND, TestPoint:TestPoint_Pad_D1.5mm, F.Cu at (152.2, 69.9)
- added TP6: +BATT, TestPoint:TestPoint_Pad_1.5x1.5mm, B.Cu at (160.0, 54.3)
- added TP7: GND, TestPoint:TestPoint_Pad_1.5x1.5mm, B.Cu at (151.9, 54.3)
- added TP8: PA1, TestPoint:TestPoint_Pad_D2.0mm, F.Cu at (139.6, 68.4)
- added U1: LT1618EDD-PBF, footprints:DFN-10_DD_LIT, F.Cu at (165.5, 56.4)
- added U2: MCP73831-2-OT, Package_TO_SOT_SMD:SOT-23-5, F.Cu at (155.9, 55.6)
- added U3: ATtiny1616-M, Package_DFN_QFN:VQFN-20-1EP_3x3mm_P0.4mm_EP1.7x1.7mm, F.Cu at (153.3, 65.5)
- J1: moved to B.Cu
- TP9: footprint footprints:TestPoint_Pad_7.0x15.0mm -> footprints:TestPoint_Pad_6.0x12.0mm; moved to B.Cu
- moved TP9 1.10 mm to (125.3, 62.9), turned to -90 degrees
- moved J1 0.64 mm to (173.6, 63.1), turned to -90 degrees
Connections:
- net /led_driver/VBUS renamed /charger/VBUS
- TP9 pad 1: /led_driver/LEDK -> GND
Routing:
- net /charger/VBUS: track 0.00 -> 40.9 mm, vias 0 -> 2
- net /mcu/USB_SBU2: track 0.00 -> 35.0 mm, vias 0 -> 4
- net +BATT: track 0.00 -> 32.4 mm, vias 0 -> 4
- net /mcu/USB_SBU1: track 0.00 -> 31.7 mm, vias 0 -> 4
- net /mcu/PC2: track 0.00 -> 25.2 mm, vias 0 -> 2
- net /mcu/PC1: track 0.00 -> 20.9 mm, vias 0 -> 2
- net /mcu/PA2: track 0.00 -> 20.5 mm, vias 0 -> 2
- net /mcu/PB3: track 0.00 -> 20.0 mm, vias 0 -> 2
- net /led_driver/nSHDN: track 0.00 -> 20.0 mm, vias 0 -> 2
- net /mcu/BTN: track 0.00 -> 18.1 mm
- net Net-(D1-K): track 0.00 -> 17.0 mm
- net /mcu/PB2: track 0.00 -> 16.7 mm, vias 0 -> 2
- net /mcu/PA1: track 0.00 -> 16.5 mm, vias 0 -> 2
- net /mcu/MCU_VCC: track 0.00 -> 16.1 mm, vias 0 -> 2
- net /charger/CHG_GATE: track 0.00 -> 12.7 mm
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- added copper zone on B.Cu, net GND
- added copper zone on F.Cu, net GND
Other:
- board text added: "0R"
- board text added: "2025-11-23"
- board text added: "BTN"
- board text added: "GND"
- board text added: "PA1"
- board text added: "PA2"
- board text added: "PB2"
- board text added: "PB3"
- board text added: "PC1"
- board text added: "PC2"
- board text added: "SBU1"
- board text added: "SBU2"
- board text added: "UPDI"
- board text added: "VCC"
- board text added: "by reykato"
- board text added: "lightwear"
- board text added: "necklace"
- board text added: "rev 0"

Commit message: small tweak
Parts:
- moved L1 0.20 mm to (173.0, 55.5)
Changed lines of the file:
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@@
 	(footprint "Inductor_SMD:L_Changjiang_FNR4030S"
 		(layer "B.Cu")
-		(at 173 55.3 90)
+		(at 173 55.5 90)
 		(descr "Inductor, Changjiang, FNR4030S, 4.0x4.0x3.0mm, (https://datasheet.lcsc.com/lcsc/1806131217_cjiang-Changjiang-Microelectronics-Tech-FNR5040S3R3NT_C167960.pdf), generated with kicad-footprint-generator gen_inductor.py")
 		(tags "wirewound power shielded")

Commit message: finishing touches made, exported as rev0
Parts:
- moved C1 28.8 mm to (169.6, 83.7)
- moved C2 28.8 mm to (166.3, 90.2)
- moved C7 28.8 mm to (171.5, 83.7)
- moved Q1 28.8 mm to (158.9, 87.9)
- moved R11 28.8 mm to (159.5, 91.7)
- moved R9 28.8 mm to (155.7, 90.4)
- moved TP9 28.8 mm to (126.0, 91.7)
- moved U1 28.8 mm to (166.2, 85.2)
- moved C4 28.8 mm to (159.6, 92.8)
- moved C5 28.8 mm to (159.6, 93.8)
- moved C6 28.8 mm to (149.7, 93.5)
- moved C8 28.8 mm to (160.9, 84.0)
- moved D1 28.8 mm to (166.3, 88.2)
- moved L1 28.8 mm to (173.8, 84.2)
- moved R1 28.8 mm to (149.7, 92.5)
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Other:
- outline, holes or cut-outs redrawn
- board text added: "+"
- board text added: "-"
