File: pcb/bracelet/lightwear_bracelet_btn_fpc/lightwear_bracelet_btn_fpc.kicad_pcb (KiCad board)
At the start: 2 copper layers, 16.9 x 9.8 mm, 3 parts, among them SW1 SW_SPST

Commit message: 20x15_audio_reactive rev0 done
Parts:
- SW1: footprint footprints:1TS016A-1800-0600-CT -> footprints:GT-TC155X-HXXXX-LX
- moved TP1 4.02 mm to (161.7, 101.3)
- moved TP2 4.02 mm to (161.7, 102.7)
- moved SW1 1.00 mm to (146.0, 102.0), turned to 0 degrees
Routing:
- net GND: track 12.4 -> 19.5 mm
- net /BTN: track 12.4 -> 19.5 mm
Other:
- board size 16.9 x 9.8 mm -> 22.5 x 11 mm
