File: pcb/bracelet/lightwear_bracelet_btn_fpc/lightwear_bracelet_btn_fpc.kicad_sch (KiCad schematic)
At the start: 3 parts, among them SW1 SW_SPST

Commit message: 20x15_audio_reactive rev0 done
Parts:
- SW1: footprint footprints:1TS016A-1800-0600-CT -> footprints:GT-TC155X-HXXXX-LX
Changed lines of the file:
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@@
 			)
 		)
-		(property "Footprint" "footprints:1TS016A-1800-0600-CT"
+		(property "Footprint" "footprints:GT-TC155X-HXXXX-LX"
 			(at 104.14 87.63 0)
 			(effects
